File: template_jsome.kicad_sch (KiCad schematic)
At the start: 8 parts

Commit message: Add files via upload
Parts:
- JSOME1_1, JSOME2_1: value Conn_01x02 -> autoremove
- JSOME22_1: value Conn_01x22 -> autoremove
- JSOME32_1: value Conn_01x32 -> autoremove
- JSOME4_1: value Conn_01x04 -> autoremove
- JSOME5_1: value Conn_01x05 -> autoremove
- JSOME6_1: value Conn_01x06 -> autoremove
- JSOME8_1: value Conn_01x08 -> autoremove
Changed lines of the file:
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@@
       (effects (font (size 1.27 1.27)) (justify left))
     )
-    (property "Value" "Conn_01x05" (at 22.86 219.71 0)
+    (property "Value" "autoremove" (at 22.86 219.71 0)
       (effects (font (size 1.27 1.27)) (justify left))
     )
@@
     (pin "4")
     (instances
-      (project "09"
+      (project "template_jsome"
         (path "/09aea597-a04d-41ef-ad99-d414ceb348c0"
           (reference "JSOME5_1") (unit 1)
@@
       (effects (font (size 1.27 1.27)) (justify left))
     )
-    (property "Value" "Conn_01x08" (at 24.13 168.91 0)
+    (property "Value" "autoremove" (at 24.13 168.91 0)
       (effects (font (size 1.27 1.27)) (justify left))
     )
@@
     (pin "8")
     (instances
-      (project "09"
+      (project "template_jsome"
         (path "/09aea597-a04d-41ef-ad99-d414ceb348c0"
           (reference "JSOME8_1") (unit 1)
@@
       (effects (font (size 1.27 1.27)) (justify left))
     )
-    (property "Value" "Conn_01x06" (at 24.13 196.85 0)
+    (property "Value" "autoremove" (at 24.13 196.85 0)
       (effects (font (size 1.27 1.27)) (justify left))
     )
@@
     (pin "6")
     (instances
-      (project "09"
+      (project "template_jsome"
         (path "/09aea597-a04d-41ef-ad99-d414ceb348c0"
           (reference "JSOME6_1") (unit 1)
@@
       (effects (font (size 1.27 1.27)) (justify left))
     )
-    (property "Value" "Conn_01x02" (at 22.86 269.24 0)
+    (property "Value" "autoremove" (at 22.86 269.24 0)
       (effects (font (size 1.27 1.27)) (justify left))
     )
@@
     (pin "1")
     (instances
-      (project "09"
+      (project "template_jsome"
         (path "/09aea597-a04d-41ef-ad99-d414ceb348c0"
           (reference "JSOME1_1") (unit 1)
@@
       (effects (font (size 1.27 1.27)) (justify left))
     )
-    (property "Value" "Conn_01x22" (at 24.13 105.41 0)
+    (property "Value" "autoremove" (at 24.13 105.41 0)
       (effects (font (size 1.27 1.27)) (justify left))
     )
@@
     (pin "11")
     (instances
-      (project "09"
+      (project "template_jsome"
         (path "/09aea597-a04d-41ef-ad99-d414ceb348c0"
           (reference "JSOME22_1") (unit 1)
@@
       (effects (font (size 1.27 1.27)) (justify left))
     )
-    (property "Value" "Conn_01x04" (at 24.13 240.03 0)
+    (property "Value" "autoremove" (at 24.13 240.03 0)
       (effects (font (size 1.27 1.27)) (justify left))
     )
@@
     (pin "1")
     (instances
-      (project "09"
+      (project "template_jsome"
         (path "/09aea597-a04d-41ef-ad99-d414ceb348c0"
           (reference "JSOME4_1") (unit 1)
@@
       (effects (font (size 1.27 1.27)) (justify left))
     )
-    (property "Value" "Conn_01x32" (at 24.13 16.51 0)
+    (property "Value" "autoremove" (at 24.13 16.51 0)
       (effects (font (size 1.27 1.27)) (justify left))
     )
@@
     (pin "31")
     (instances
-      (project "09"
+      (project "template_jsome"
         (path "/09aea597-a04d-41ef-ad99-d414ceb348c0"
           (reference "JSOME32_1") (unit 1)
@@
       (effects (font (size 1.27 1.27)) (justify left))
     )
-    (property "Value" "Conn_01x02" (at 22.86 257.81 0)
+    (property "Value" "autoremove" (at 22.86 257.81 0)
       (effects (font (size 1.27 1.27)) (justify left))
     )
@@
     (pin "1")
     (instances
-      (project "09"
+      (project "template_jsome"
         (path "/09aea597-a04d-41ef-ad99-d414ceb348c0"
           (reference "JSOME2_1") (unit 1)

Commit message: Add files via upload
Parts:
- added JSOME0_1: autoremove, Symbol:OSHW-Symbol_6.7x6mm_SilkScreen, symbol Connector_Generic:Conn_01x02
Changed lines of the file:
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@@
 (kicad_sch (version 20230121) (generator eeschema)
   (paper "A4")
+  (symbol (lib_id "Connector_Generic:Conn_01x02") (at 17.78 283.21 0) (mirror y) (unit 1)
+    (in_bom yes) (on_board yes) (dnp no)
+    (property "Reference" "JSOME0_1" (at 21.59 278.13 0)
+      (effects (font (size 1.27 1.27)) (justify left))
+    )
+    (property "Value" "autoremove" (at 22.86 280.67 0)
+      (effects (font (size 1.27 1.27)) (justify left))
+    )
+    (property "Footprint" "Symbol:OSHW-Symbol_6.7x6mm_SilkScreen" (at 17.78 283.21 0)
+      (effects (font (size 1.27 1.27)) hide)
+    )
+    (property "Datasheet" "~" (at 17.78 283.21 0)
+      (effects (font (size 1.27 1.27)) hide)
+    )
+    (pin "2")
+    (pin "1")
+    (instances
+      (project "template_jsome"
+        (path "/09aea597-a04d-41ef-ad99-d414ceb348c0"
+          (reference "JSOME0_1") (unit 1)
+        )
+      )
+    )
+  )
   (symbol (lib_id "Connector_Generic:Conn_01x05") (at 17.78 228.6 0) (mirror y) (unit 1)
     (in_bom yes) (on_board yes) (dnp no)
