File: freeeeg8-alpha.kicad_sch (KiCad schematic)
At the start: 35 parts, among them J1 AIN0, J10 GND, J12 STACK_1, J13 STACK_2, J14 XIAO_1, J15 XIAO_2, J2 AIN1, J3 AIN2, J4 AIN3, J5 AIN4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

Commit message: Add files via upload
Parts:
- C1: MPN (none) -> CC0402KRX5R5BB224
- C2: MPN (none) -> CL05B104KO5NNNC
- C3, C4: MPN (none) -> CL05A105KO5NNNC
- C5, C6, C7, C8: MPN (none) -> GRM188R71A225KE15D
- J1, J10, J2, J3, J4, J5, J6, J7, J8, J9: MPN (none) -> pogo-pin-d5x10mm-smd
- J12, J13: MPN (none) -> 53398-0671
- J14, J15: MPN (none) -> TSM-107-01-L-SV
- R1, R2, R3, R4: MPN (none) -> RC0402JR-070RL
- R5: MPN (none) -> DNP
- U1: MPN (none) -> ADS131M08IPBSR
- U2, U3: MPN (none) -> LP5907QMFX-3.3Q1
- X1: MPN (none) -> ECS-2520MVLC-081.92-CN-TR

Commit message: Add files via upload
Connections:
- net AINREF_STACK: now also J12.2 (Pin_2), J13.5 (Pin_5); no longer J12.3 (Pin_3), J13.4 (Pin_4)
- net DIN: now also J15.3 (Pin_3); no longer J15.5 (Pin_5)
- net SCLK: now also J15.5 (Pin_5); no longer J15.3 (Pin_3)
- net SYNC/RESET_ADC: now also J12.4 (Pin_4), J13.3 (Pin_3); no longer J12.2 (Pin_2), J13.5 (Pin_5)
- net XTAL1/CLKIN: now also J12.3 (Pin_3), J13.4 (Pin_4); no longer J12.4 (Pin_4), J13.3 (Pin_3)
Changed lines of the file:
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@@
 	)
 	(label "DIN"
-		(at 143.51 34.29 0)
+		(at 143.51 29.21 0)
 		(effects
 			(font
@@
 	)
 	(label "SCLK"
-		(at 143.51 29.21 0)
+		(at 143.51 34.29 0)
 		(effects
 			(font
@@
 	)
 	(label "XTAL1/CLKIN"
-		(at 88.9 88.9 0)
+		(at 88.9 86.36 0)
 		(effects
 			(font
@@
 	)
 	(label "AINREF_STACK"
-		(at 121.92 88.9 0)
+		(at 121.92 91.44 0)
 		(effects
 			(font
@@
 	)
 	(label "AINREF_STACK"
-		(at 88.9 86.36 0)
+		(at 88.9 83.82 0)
 		(effects
 			(font
@@
 	)
 	(label "SYNC/RESET_ADC"
-		(at 88.9 83.82 0)
+		(at 88.9 88.9 0)
 		(effects
 			(font
@@
 	)
 	(label "SYNC/RESET_ADC"
-		(at 121.92 91.44 0)
+		(at 121.92 86.36 0)
 		(effects
 			(font
@@
 	)
 	(label "XTAL1/CLKIN"
-		(at 121.92 86.36 0)
-		(effects
-			(font
+		(at 121.92 88.9 0)
+		(effects
+			(font

Commit message: Add files via upload
Parts:
- R5: DNP (none) -> DNP
Connections:
- net CS: now also U4.5 (Pin_5); no longer U4.3 (Pin_3)
- net DIN: now also U4.10 (Pin_10); no longer U4.11 (Pin_11)
- net DOUT: now also U4.11 (Pin_11); no longer U4.10 (Pin_10)
- net DRDY: now also U4.6 (Pin_6); no longer U4.2 (Pin_2)
- net SCLK: now also U4.12 (Pin_12); no longer U4.9 (Pin_9)
- net SYNC/RESET_XIAO: now also U4.4 (Pin_4); no longer U4.1 (Pin_1)
- net XIAO_NC1: now also U4.1 (Pin_1); no longer U4.4 (Pin_4)
- net XIAO_NC2: now also U4.2 (Pin_2); no longer U4.5 (Pin_5)
- net XIAO_NC3: now also U4.3 (Pin_3); no longer U4.6 (Pin_6)
- net XIAO_NC6: now also U4.9 (Pin_9); no longer U4.12 (Pin_12)
Changed lines of the file:
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@@
 		)
 	)
-	(label "CS"
-		(at 50.8 30.48 0)
+	(label "XIAO_NC1"
+		(at 50.8 25.4 0)
 		(effects
 			(font
@@
 		)
 	)
-	(label "XIAO_NC1"
-		(at 50.8 33.02 0)
-		(effects
-			(font
-				(size 1.27 1.27)
-			)
-			(justify left bottom)
-		)
-	)
 	(label "DVDD"
 		(at 40.65 187.96 0)
@@
 		)
 	)
-	(label "BAT+"
-		(at 50.8 78.74 0)
+	(label "CS"
+		(at 50.8 35.56 0)
 		(effects
 			(font
@@
 		)
 	)
-	(label "AINREF"
-		(at 100.65 187.96 0)
+	(label "SYNC/RESET_XIAO"
+		(at 50.8 33.02 0)
 		(effects
 			(font
@@
 		)
 	)
-	(label "SCLK"
-		(at 143.51 34.29 0)
+	(label "BAT+"
+		(at 50.8 78.74 0)
 		(effects
 			(font
@@
 		)
 	)
-	(label "XIAO_NC3"
-		(at 50.8 38.1 0)
+	(label "AINREF"
+		(at 100.65 187.96 0)
+		(effects
+			(font
+				(size 1.27 1.27)
+			)
+			(justify left bottom)
+		)
+	)
+	(label "SCLK"
+		(at 143.51 34.29 0)
 		(effects
 			(font
@@
 	)
 	(label "XIAO_NC6"
-		(at 50.8 53.34 0)
+		(at 50.8 45.72 0)
 		(effects
 			(font
@@
 		)
 	)
+	(label "DRDY"
+		(at 50.8 38.1 0)
+		(effects
+			(font
+				(size 1.27 1.27)
+			)
+			(justify left bottom)
+		)
+	)
 	(label "AINREF_STACK"
 		(at 121.92 91.44 0)
@@
 	)
 	(label "SCLK"
-		(at 50.8 45.72 0)
+		(at 50.8 53.34 0)
 		(effects
 			(font
@@
 		)
 	)
-	(label "DRDY"
-		(at 50.8 27.94 0)
-		(effects
-			(font
-				(size 1.27 1.27)
-			)
-			(justify left bottom)
-		)
-	)
 	(label "AINREF_POGOPIN"
 		(at 190.82 152.4 0)
@@
 	)
 	(label "DIN"
-		(at 50.8 50.8 0)
+		(at 50.8 48.26 0)
 		(effects
 			(font
@@
 		)
 	)
+	(label "XIAO_NC3"
+		(at 50.8 30.48 0)
+		(effects
+			(font
+				(size 1.27 1.27)
+			)
+			(justify left bottom)
+		)
+	)
 	(label "NFC1"
 		(at 70.8 104.14 0)
@@
 		)
 	)
-	(label "SYNC/RESET_XIAO"
-		(at 50.8 25.4 0)
-		(effects
-			(font
-				(size 1.27 1.27)
-			)
-			(justify left bottom)
-		)
-	)
 	(label "GND"
 		(at 50.8 55.88 0)
@@
 		)
 	)
-	(label "5V"
-		(at 121.92 81.28 0)
+	(label "XIAO_NC2"
+		(at 50.8 27.94 0)
 		(effects
 			(font
@@
 		)
 	)
-	(label "XIAO_NC2"
-		(at 50.8 35.56 0)
+	(label "5V"
+		(at 121.92 81.28 0)
 		(effects
 			(font
@@
 	)
 	(label "DOUT"
-		(at 50.8 48.26 0)
+		(at 50.8 50.8 0)
 		(effects
 			(font
@@
 			(at 86.36 173.99 0)
 			(effects
+				(font
+					(size 1.27 1.27)
+				)
+				(hide yes)
+			)
+		)
+		(property "DNP" "DNP"
+			(at 86.36 173.99 0)
+			(effects

Commit message: Add files via upload
Connections:
- net XIAO_NC6 is gone; now on net DIN: J15.2 (Pin_2), U4.9 (Pin_9)
- net DIN: no longer J15.3 (Pin_3), U4.10 (Pin_10)
- net DOUT: now also J15.3 (Pin_3), U4.10 (Pin_10); no longer J15.4 (Pin_4), U4.11 (Pin_11)
- net SCLK: now also J15.4 (Pin_4), U4.11 (Pin_11); no longer J15.5 (Pin_5), U4.12 (Pin_12)
- new net 3_3V: J15.5 (Pin_5), U4.12 (Pin_12)
Changed lines of the file:
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@@
 	)
 	(label "DIN"
-		(at 143.51 29.21 0)
+		(at 50.8 45.72 0)
 		(effects
 			(font
@@
 		)
 	)
+	(label "SCLK"
+		(at 50.8 50.8 0)
+		(effects
+			(font
+				(size 1.27 1.27)
+			)
+			(justify left bottom)
+		)
+	)
 	(label "BAT+"
 		(at 50.8 78.74 0)
@@
 		)
 	)
-	(label "SCLK"
-		(at 143.51 34.29 0)
-		(effects
-			(font
-				(size 1.27 1.27)
-			)
-			(justify left bottom)
-		)
-	)
 	(label "SYNC/RESET_XIAO"
 		(at 115.57 29.21 0)
@@
 		)
 	)
-	(label "XIAO_NC6"
-		(at 50.8 45.72 0)
-		(effects
-			(font
-				(size 1.27 1.27)
-			)
-			(justify left bottom)
-		)
-	)
 	(label "GND"
 		(at 80.65 187.96 0)
@@
 		)
 	)
+	(label "SCLK"
+		(at 143.51 31.75 0)
+		(effects
+			(font
+				(size 1.27 1.27)
+			)
+			(justify left bottom)
+		)
+	)
 	(label "GND"
 		(at 70.8 93.98 0)
@@
 		)
 	)
-	(label "SCLK"
-		(at 50.8 53.34 0)
-		(effects
-			(font
-				(size 1.27 1.27)
-			)
-			(justify left bottom)
-		)
-	)
 	(label "AIN6P"
 		(at 25.4 44.45 0)
@@
 		)
 	)
-	(label "DOUT"
-		(at 143.51 31.75 0)
-		(effects
-			(font
-				(size 1.27 1.27)
-			)
-			(justify left bottom)
-		)
-	)
 	(label "5V"
 		(at 50.8 58.42 0)
@@
 		)
 	)
-	(label "XIAO_NC6"
-		(at 143.51 26.67 0)
-		(effects
-			(font
-				(size 1.27 1.27)
-			)
-			(justify left bottom)
-		)
-	)
 	(label "DVDD"
 		(at 95.25 36.83 0)
@@
 		)
 	)
+	(label "DOUT"
+		(at 143.51 29.21 0)
+		(effects
+			(font
+				(size 1.27 1.27)
+			)
+			(justify left bottom)
+		)
+	)
 	(label "SWCLK"
 		(at 70.8 96.52 0)
@@
 		)
 	)
+	(label "DIN"
+		(at 143.51 26.67 0)
+		(effects
+			(font
+				(size 1.27 1.27)
+			)
+			(justify left bottom)
+		)
+	)
+	(label "3_3V"
+		(at 50.8 53.34 0)
+		(effects
+			(font
+				(size 1.27 1.27)
+			)
+			(justify left bottom)
+		)
+	)
 	(label "GND"
 		(at 211.13 134.62 0)
@@
 		)
 	)
-	(label "DIN"
-		(at 50.8 48.26 0)
-		(effects
-			(font
-				(size 1.27 1.27)
-			)
-			(justify left bottom)
-		)
-	)
 	(label "AIN4P"
 		(at 110.82 152.4 0)
@@
 		)
 	)
+	(label "DOUT"
+		(at 50.8 48.26 0)
+		(effects
+			(font
+				(size 1.27 1.27)
+			)
+			(justify left bottom)
+		)
+	)
 	(label "AINREF"
 		(at 91.44 176.53 0)
@@
 		)
 	)
+	(label "3_3V"
+		(at 143.51 34.29 0)
+		(effects
+			(font
+				(size 1.27 1.27)
+			)
+			(justify left bottom)
+		)
+	)
 	(label "GND"
 		(at 50.8 55.88 0)
@@
 		(effects
 			(font
-				(size 1.27 1.27)
-			)
-			(justify left bottom)
-		)
-	)
-	(label "DOUT"
-		(at 50.8 50.8 0)
-		(effects
-			(font
