File: freeeeg8-alpha.kicad_pcb (KiCad board)
At the start: 2 copper layers, 26 x 26 mm, 33 parts, among them J1 AIN0, J10 GND, J12 STACK_1, J13 STACK_2, J14 XIAO_1, J15 XIAO_2, J2 AIN1, J3 AIN2, J4 AIN3, J5 AIN4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

Commit message: Add files via upload
Parts:
- moved R5 5.46 mm to (5.59, -4.95)
- moved C7 1.63 mm to (4.83, 0.76), turned to 180 degrees
- moved C5 1.37 mm to (-5.33, 0.89), turned to 180 degrees
- moved C2 1.02 mm to (-4.70, -1.40)
- moved R4 0.92 mm to (10.5, -2.41)
- moved C4 0.89 mm to (4.70, -1.27)
- moved R1 0.68 mm to (10.5, 1.91)
- moved C3 0.65 mm to (-3.30, 0.89)
- moved R2 0.64 mm to (-10.8, -1.91)
- moved C8 0.25 mm to (6.10, 5.08)
- moved J14 0.13 mm to (-8.51, 0.00)
- moved J15 0.13 mm to (8.51, 0.00)
- moved X1 0.05 mm to (0.00, 4.14)
Connections:
- J12 pad 2: /SYNC/RESET_ADC -> /AINREF_STACK
- J12 pad 3: /AINREF_STACK -> /XTAL1/CLKIN
- J12 pad 4: /XTAL1/CLKIN -> /SYNC/RESET_ADC
- J13 pad 3: /XTAL1/CLKIN -> /SYNC/RESET_ADC
- J13 pad 4: /AINREF_STACK -> /XTAL1/CLKIN
- J13 pad 5: /SYNC/RESET_ADC -> /AINREF_STACK
- J15 pad 3: /SCLK -> /DIN
- J15 pad 5: /DIN -> /SCLK
Routing:
- net /AINREF: track 25.6 -> 47.6 mm, vias 5 -> 0
- net /5V: track 72.2 -> 87.4 mm
- net /AINREF_STACK: track 29.6 -> 21.3 mm, vias 3 -> 2
- net /GND: track 104.9 -> 112.9 mm, vias 0 -> 19
- net /XTAL1/CLKIN: track 21.5 -> 28.3 mm
- net /AIN0P: track 21.2 -> 16.3 mm
- net /AINREF_POGOPIN: track 1.85 -> 5.05 mm
- net /CS: track 9.72 -> 12.7 mm, vias 2 -> 0
- net /SYNC/RESET_ADC: track 38.9 -> 36.7 mm, vias 5 -> 3
- net /AIN6P: track 15.5 -> 13.4 mm
- net /DRDY: track 7.32 -> 9.42 mm, vias 2 -> 0
- net /AVDD: track 8.82 -> 7.08 mm
- net /AIN7P: track 17.4 -> 15.7 mm
- net /AIN4P: track 7.97 -> 9.58 mm
- net /SCLK: track 14.3 -> 12.7 mm
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
Commit message: Add files via upload
Parts:
- J12, J13: footprint freeeeg8-alpha:Molex_PicoBlade_53398-0671_1x06-1MP_P1.25mm_Vertical -> freeeeg8-alpha:Molex_PicoBlade_53398-0671_1x06-1MP_P1.25mm_Vertical_round_cut
Routing:
- net /AINREF: track 47.6 -> 37.8 mm

Commit message: Add files via upload
Parts:
- moved C2 0.09 mm to (-4.69, -1.31)
- moved X1 0.07 mm to (0.00, 4.21)
Routing:
- net /AINREF: track 37.8 -> 23.8 mm
- net /AINREF_STACK: track 21.3 -> 24.1 mm
- net /GND_POGOPIN: track 3.97 -> 1.26 mm
- net /CS: track 12.7 -> 10.3 mm
- net /5V: track 87.4 -> 89.8 mm
- net /AIN1P: track 16.4 -> 17.9 mm
- net /AIN0P: track 16.3 -> 17.7 mm
- net /SYNC/RESET_ADC: track 36.7 -> 38.1 mm
- net /GND: track 113.2 -> 112.3 mm, vias 19 -> 18
- net /SCLK: track 12.7 -> 11.8 mm
- net /DOUT: track 13.6 -> 12.9 mm
- net /XTAL1/CLKIN: track 28.4 -> 29.0 mm
- net /AVDD: track 7.08 -> 7.21 mm, vias 0 -> 2

Commit message: Add files via upload
Routing:
- net /GND: track 112.3 -> 116.4 mm, vias 18 -> 19
- net /AINREF_POGOPIN: track 4.97 -> 2.49 mm
- net /AINREF: track 23.8 -> 24.8 mm
- net /SCLK: track 11.8 -> 12.6 mm
- net /DOUT: track 12.9 -> 13.7 mm
- net /AIN7P: track 15.8 -> 16.6 mm
- net /AINREF_STACK: track 24.1 -> 23.4 mm
- net /AIN4P: track 9.15 -> 9.84 mm
- net /DRDY: track 8.96 -> 9.64 mm

Commit message: Add files via upload
Connections:
- J15 pad 2: /XIAO_NC6 -> /DIN
- J15 pad 3: /DIN -> /DOUT
- J15 pad 4: /DOUT -> /SCLK
- J15 pad 5: /SCLK -> /3_3V
Routing:
- net /DIN: track 10.3 -> 16.5 mm
- net /DOUT: track 13.7 -> 10.8 mm
- net /SCLK: track 12.6 -> 15.5 mm
- net /GND: track 116.4 -> 117.9 mm
- net /DVDD: track 15.4 -> 16.0 mm

Commit message: Add files via upload
Parts:
- J14, J15: footprint Connector_PinHeader_2.54mm:PinHeader_1x07_P2.54mm_Vertical_SMD_Pin1Right -> Connector_PinSocket_2.54mm:PinSocket_1x07_P2.54mm_Vertical_SMD_Pin1Right
- X1: footprint freeeeg8-alpha:Oscillator_SMD_EuroQuartz_XO32-4Pin_3.2x2.5mm_HandSoldering -> freeeeg8-alpha:Oscillator_SMD_EuroQuartz_XO32-4Pin_3.2x2.5mm_HandSoldering_short
Routing:
- net /GND: track 117.9 -> 119.0 mm
