File: freeeeg8-alpha.kicad_pcb (KiCad board)
At the start: 2 copper layers, 26 x 26 mm, 33 parts, among them J1 AIN0, J10 GND, J12 STACK_1, J13 STACK_2, J14 XIAO_1, J15 XIAO_2, J2 AIN1, J3 AIN2, J4 AIN3, J5 AIN4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

Commit message: Add files via upload
Parts:
- moved R5 5.92 mm to (10.9, -2.31)
- moved R4 2.01 mm to (10.9, -0.44)
- moved J14 0.89 mm to (-7.62, 0.00)
- moved J15 0.89 mm to (7.62, 0.00)
- moved C5 0.81 mm to (-4.61, 1.25)
- moved C3 0.77 mm to (-2.54, 0.97)
- moved C8 0.58 mm to (5.53, 4.98)
- moved C2 0.55 mm to (-5.15, -1.00)
- moved C6 0.54 mm to (-5.56, 4.90)
- moved R1 0.36 mm to (10.9, 1.90)
- moved C4 0.30 mm to (4.82, -1.00)
- moved C7 0.25 mm to (4.73, 1.00)
- moved GL1 0.05 mm to (0.00, -12.5)
- turned R2 to -90 degrees
Routing:
- net /SYNC/RESET_ADC: track 38.3 -> 30.1 mm
- net /AINREF_STACK: track 23.4 -> 29.9 mm
- net /GND: track 119.0 -> 114.5 mm
- net /XTAL1/CLKIN: track 29.0 -> 25.5 mm
- net /CS: track 10.2 -> 8.30 mm
- net (no net): track 0.00 -> 1.91 mm, vias 0 -> 4
- net /AIN7P: track 16.6 -> 18.3 mm, vias 1 -> 2
- net /5V: track 89.7 -> 88.2 mm, vias 0 -> 1
- net /AIN1P: track 17.8 -> 19.3 mm, vias 1 -> 2
- net /AIN2P: track 7.11 -> 8.52 mm, vias 1 -> 2
- net /AINREF_POGOPIN: track 2.49 -> 1.18 mm
- net /AIN6P: track 13.3 -> 14.6 mm, vias 1 -> 2
- net /DRDY: track 9.64 -> 8.42 mm
- net /AIN5P: track 7.10 -> 8.21 mm, vias 1 -> 2
- net /AINREF: track 24.8 -> 25.9 mm
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